Commit message: adjusted urdf, added dummy link

File: config/urdf/sensor_traeger_base.xacro (robot description, xacro)
@@ -3,5 +3,15 @@
     <xacro:property name="nav_length" value="1.2" />
     <xacro:property name="nav_width" value="0.1"/>
+    <link name="dummy"/>
+    <joint name="dummyjoint" type="fixed">
+        <parent link="dummy"/>
+        <child link="base_link"/>
+        <origin xyz="0 0 0" rpy= "0 0 0"/>
+    </joint>
     <link name="base_link">
+        <!-- <xacro:box_inertia m="0.5" l="${nav_length}" w="${nav_width}" h="${nav_width}" -->
+                           <!-- xyz="0 0 ${nav_width / 2}" rpy="0 0 0" /> -->
+    </link>
+    <link name="gps_link">
         <visual>
             <geometry>
@@ -17,8 +27,4 @@
             <origin xyz="0 0 ${nav_width / 2}" rpy="0 0 0"/>
         </collision>
-        <!-- <xacro:box_inertia m="0.5" l="${nav_length}" w="${nav_width}" h="${nav_width}" -->
-                           <!-- xyz="0 0 ${nav_width / 2}" rpy="0 0 0" /> -->
-    </link>
-    <link name="gps_link">
     </link>
     <link name="imu_link">
@@ -42,5 +48,5 @@
         <parent link="base_link"/>
         <child link="imu_link"/>
-        <origin xyz="0 0 ${nav_width}" rpy= "0 0 0"/>
+        <origin xyz="0 -0.17 ${nav_width}" rpy= "0 0 0"/>
     </joint>
     <xacro:macro name="gps_link" params="prefix">
@@ -78,5 +84,5 @@
         <parent link="base_link"/>
         <child link="gps_link"/>
-        <origin xyz="0 0 0" rpy= "0 0 0"/>
+        <origin xyz="0 -0.17 0" rpy= "0 0 0"/>
     </joint>
 </robot>
